Commit message: debugging stand up state

File: DARoS-Ctrl/Systems/PrestoeSystem/Robot/prestoe_urdf.urdf (robot description, URDF)
Before this commit: robot prestoe, 24 links, 23 joints
Joints:
- joint L_hipyaw: origin xyz=0 54.71371e-3 -48.37244e-3 rpy=0.2618  0  0 -> xyz=0 54.71371e-3 -48.37244e-3 rpy=0.2618 0 0
- joint R_hipyaw: origin xyz=0 -54.71371e-3 -48.37244e-3 rpy=-0.2618  0  0 -> xyz=0 -54.71371e-3 -48.37244e-3 rpy=-0.2618 0 0

Commit message: link, joint, contact point index adjustment

File: DARoS-Ctrl/Systems/PrestoeSystem/Robot/prestoe_urdf.urdf (robot description, URDF)
Before this commit: robot prestoe, 24 links, 23 joints
Joints:
- removed joint L_hipyaw
- removed joint L_shoulderpitch
- removed joint R_hipyaw
- removed joint R_shoulderpitch
- removed joint torsoyaw
- added joint a_torsoyaw: type revolute, parent torso_link, child pelvis, origin xyz=0.0 0.0 -44.5e-3 rpy=0 0 0, axis 0 0 1, limit lower=-1.57079632679 upper=1.57079632679 effort=1000 velocity=20
- added joint bR_hipyaw: type revolute, parent pelvis, child R_hipyaw_link, origin xyz=0 -54.71371e-3 -48.37244e-3 rpy=-0.2618 0 0, axis 0 0 1, limit lower=-1.57 upper=1.57 effort=0.0 velocity=20.0
- added joint cL_hipyaw: type revolute, parent pelvis, child L_hipyaw_link, origin xyz=0 54.71371e-3 -48.37244e-3 rpy=0.2618 0 0, axis 0 0 1, limit lower=-1.570796 upper=1.570796 effort=100 velocity=20
- added joint yR_shoulderpitch: type revolute, parent torso_link, child R_shoulderpitch_link, origin xyz=0 -106.840e-3 300.24519e-3 rpy=1.1345 0 0, axis 0 0 1, limit lower=-2.61799387799 upper=0.9 effort=100 velocity=20
- added joint zL_shoulderpitch: type revolute, parent torso_link, child L_shoulderpitch_link, origin xyz=0 106.840e-3 300.24519e-3 rpy=-1.1345 0 0, axis 0 1 0, limit lower=-2.61799387799 upper=0.9 effort=100 velocity=20

Commit message: fixed bug in urdf - l shoulder pitch is set by y axis

File: DARoS-Ctrl/Systems/PrestoeSystem/Robot/prestoe_urdf.urdf (robot description, URDF)
Before this commit: robot prestoe, 24 links, 23 joints
Joints:
- joint zL_shoulderpitch: axis 0 1 0 -> 0 0 1
